File: KiCad/ecal_simple_solt.kicad_sch (KiCad schematic)
At the start: 18 parts, among them J1 PORT1, J2 PORT2, J3 GPIO, U1 BGS14PN10, U2 BGS14PN10, U3 BGS12PN10, U4 BGS12PN10

Commit message: New revision
Parts:
- removed J3: GPIO, Infineon:PinHeader_2x10_P2.54mm_Horizontal_SMD, symbol Connector_Generic:Conn_02x10_Odd_Even
- removed U3, U4: BGS12PN10, Infineon:XQFP-10, symbol Infineon:BGS12PN10
- added H1, H2, H3, H4: MountingHole, MountingHole:MountingHole_3.2mm_M3_ISO7380, symbol Mechanical:MountingHole
- added J10: S4C1, Infineon:CPG-01-TH-B, symbol Connector_Generic:Conn_01x01
- added J11: S4C2, Infineon:CPG-01-TH-B, symbol Connector_Generic:Conn_01x01
- added J12, J13, J14, J16: GND, Infineon:CPG-01-TH-B, symbol Connector_Generic:Conn_01x01
- added J15: 3V3, Infineon:CPG-01-TH-B, symbol Connector_Generic:Conn_01x01
- added J17, J18: HEAT, Infineon:CPG-01-TH-B, symbol Connector_Generic:Conn_01x01
- added J3: THERM, Infineon:CPG-01-TH-B, symbol Connector_Generic:Conn_01x01
- added J4: S1C1, Infineon:CPG-01-TH-B, symbol Connector_Generic:Conn_01x01
- added J5: S1C2, Infineon:CPG-01-TH-B, symbol Connector_Generic:Conn_01x01
- added J6: S2C1, Infineon:CPG-01-TH-B, symbol Connector_Generic:Conn_01x01
- added J7: S2C2, Infineon:CPG-01-TH-B, symbol Connector_Generic:Conn_01x01
- added J8: S3C1, Infineon:CPG-01-TH-B, symbol Connector_Generic:Conn_01x01
- added J9: S3C2, Infineon:CPG-01-TH-B, symbol Connector_Generic:Conn_01x01
- added TH1: 10k, Resistor_SMD:R_0402_1005Metric, symbol Device:Thermistor_NTC
- added TP1, TP2: TestPoint, TestPoint:TestPoint_Pad_1.0x1.0mm, symbol Connector:TestPoint
- added U3, U4: BGS14PN10, Infineon:XQFP-10, symbol Infineon:BGS14PN10
- C1, C2, C3, C4: value C -> 100n
- J1, J2: footprint Infineon:1092-03A-6 -> Infineon:32K243-40ML5; MPN (none) -> 32K243-40ML5; Mouser No (none) -> 476-32K243-40ML5
- R101, R102: value 300 -> 292
- R103: value 18 -> 17.6
- R11, R12, R21, R22: value 100 -> 100 0.1%; footprint Resistor_SMD:R_0402_1005Metric -> Resistor_SMD:R_0201_0603Metric
- U1, U2: MPN (none) -> BGS14PN10E6327XTSA1; Mouser No (none) -> 726-BGS14PN10E6327X
Connections:
- net +3V3: now also J15.1 (Pin_1), U3.4 (VDD), U4.4 (VDD)
- net GND: now also J12.1 (Pin_1), J13.1 (Pin_1), J14.1 (Pin_1), J16.1 (Pin_1), TH1.2, U3.2 (GND), U3.7 (RF4), U3.8 (GND), U4.2 (GND), U4.7 (RF4), U4.8 (GND)
- net SW1_3dB: now also U3.1 (RF1)
- net SW1_CTRL1: now also J4.1 (Pin_1)
- net SW1_CTRL2: now also J5.1 (Pin_1)
- net SW1_Through: now also U3.10 (RFC)
- net SW2_3dB: now also U4.9 (RF3)
- net SW2_CTRL1: now also J6.1 (Pin_1)
- net SW2_CTRL2: now also J7.1 (Pin_1)
- net SW2_Through: now also U4.10 (RFC)
- net SW_Through: now also U3.9 (RF3), U4.1 (RF1)
- new net HEAT: J17.1 (Pin_1), J18.1 (Pin_1), TP1.1, TP2.1
- new net SW3_CTRL1: J8.1 (Pin_1), U3.5 (CTRL1)
- new net SW3_CTRL2: J9.1 (Pin_1), U3.6 (CTRL2)
- new net SW4_CTRL1: J10.1 (Pin_1), U4.5 (CTRL1)
- new net SW4_CTRL2: J11.1 (Pin_1), U4.6 (CTRL2)
- new net THERM: J3.1 (Pin_1), TH1.1
- no-connect marks 2 -> 4
Other:
- note added: "5%: 300 Ohm, 18 Ohm 2%: 287 Ohm, 17.8 Ohm 1%: 294 Ohm, 17.8 Ohm 0.5%: 291 Ohm, 17.6 Ohm"
- moved on the sheet: C4
