File: KiCad/ecal_simple_solt/ecal_simple_solt.kicad_pcb (KiCad board)
At the start: 4 copper layers, 30 x 35.6 mm, 40 parts, among them J1 PORT1, J10 S4C1, J11 S4C2, J12 GND, J13 GND, J14 GND, J15 3V3, J16 GND, J17 HEAT, J18 HEAT, J2 PORT2, J3 THERM, J4 S1C1, J5 S1C2, J6 S2C1, J7 S2C2, J8 S3C1, J9 S3C2, U1 BGS14PN10, U2 BGS14PN10, U3 BGS14PN10, U4 BGS14PN10

Commit message: Better directory structure
Parts:
- R101, R102: value 300 -> 292
- R103: value 18 -> 17.6
- R11, R12, R21, R22: value 100 -> 100 0.1%
Routing:
- net /HEAT: track 870.0 -> 734.6 mm

Commit message: Bit of an overdue commit
Parts:
- moved J17 1.10 mm to (94.5, 61.7)
- moved J18 1.10 mm to (89.5, 61.7)
- moved J10 0.90 mm to (97.0, 64.7)
- moved J11 0.90 mm to (94.5, 64.7)
- moved J14 0.90 mm to (99.5, 64.7)
- moved J15 0.90 mm to (92.0, 64.7)
- moved J16 0.90 mm to (84.5, 64.7)
- moved J8 0.90 mm to (89.5, 64.7)
- moved J9 0.90 mm to (87.0, 64.7)
- moved TP1 0.90 mm to (81.0, 64.7)
- moved TP2 0.90 mm to (103.0, 64.7)
Routing:
- net SW4_CTRL2: track 9.76 -> 10.7 mm
- net SW3_CTRL1: track 8.94 -> 9.84 mm
- net +3V3: track 38.9 -> 39.6 mm
- net /HEAT: track 734.6 -> 735.2 mm
